File: PCB_USB_TTL/PCB_USB_TTL.kicad_sch (KiCad schematic)
At the start: 24 parts, among them J1 Conn_01x03_Male, J2 Conn_01x06_Male, J3 Conn_01x02_Male, J4 Conn_01x02_Male, P1 USB_C_Plug, Q1 BC817, Q2 BC817, U1 AZ1117H-3.3TRE1, U2 CH340G

Commit message: Rev 2
Switch is added to change from 3.3v to 5v.

UMH3N is used to save space and cost.
Parts:
- removed J1: Conn_01x03_Male, Connector_PinHeader_2.54mm:PinHeader_1x03_P2.54mm_Vertical, symbol Connector:Conn_01x03_Male
- removed Q1, Q2: BC817, Package_TO_SOT_SMD:SOT-23, symbol Transistor_BJT:BC817
- removed R1, R2: 1K, Resistor_SMD:R_1206_3216Metric_Pad1.30x1.75mm_HandSolder, symbol Device:R
- removed U2: CH340G, Package_SO:SOIC-16_3.9x9.9mm_P1.27mm, symbol Interface_USB:CH340G
- added Q3: UMH3N, Package_TO_SOT_SMD:SOT-363_SC-70-6, symbol Transistor_BJT:UMH3N
- added SW1: ~, JAPS:MS-22D28-G020, symbol JAPS:MS-22D28-G020
- added U3: CH340C, Package_SO:SOIC-16_3.9x9.9mm_P1.27mm, symbol Interface_USB:CH340C
- R3: value 220 -> 1K
Connections:
- net +3.3V: now also SW1.6
- net +5V: now also SW1.4
- net D+: now also U3.5 (UD+)
- net D-: now also U3.6 (UD-)
- net DTR: now also Q3.2 (B1), Q3.3 (C2), U3.13 (~{DTR})
- net ESP_IO0: now also Q3.4 (E2)
- net GND: now also U3.1 (GND)
- net RTS: now also Q3.1 (E1), Q3.5 (B2), U3.14 (~{RTS})
- net VCC: now also SW1.5, U3.16 (VCC)
- net at R5.1: now also U3.3 (RXD)
- net at R4.1: now also U3.2 (TXD)
- net at C2.2: now also U3.4 (V3)
- net ESP_EN renamed REST
- net REST: now also Q3.6 (C1)
- no-connect marks 17 -> 15
Other:
- company: (none) -> Softver
- title: (none) -> USB to TTL Adapter
